Commit message: - Ajustes no panda_config para execução do moveit com o Panda robot     - Alteração direto no arquivo /panda_moveit_config/config/panda_gazebo.urdf     (gerado pelo MSA)     - FOram removidas duplicatas de controladores     - Controladores tipo effort não funcionaram (não moviam o braço),     controladores do tipo position movimentaram o braço     - Arquivo ros_controllers.yaml foi corrigido para controladores     do tipo position

File: catkin_ws/src/panda_moveit_config/config/gazebo_panda.urdf (robot description, URDF)
Before this commit: robot panda, 22 links, 21 joints
Links:
- added link world
- link panda_hand: mass 0.1 -> 0.73
- link panda_hand_sc: mass 0.1 -> None; geometry 
- link panda_leftfinger: mass 0.1 -> 0.015
- link panda_link0: mass 0.1 -> 0.629769
- link panda_link0_sc: mass 0.1 -> None; geometry 
- link panda_link1: mass 0.1 -> 4.970684
- link panda_link1_sc: mass 0.1 -> None; geometry 
- link panda_link2: mass 0.1 -> 0.646926
- link panda_link2_sc: mass 0.1 -> None; geometry 
- link panda_link3: mass 0.1 -> 3.228604
- link panda_link3_sc: mass 0.1 -> None; geometry 
- link panda_link4: mass 0.1 -> 3.587895
- link panda_link4_sc: mass 0.1 -> None; geometry 
- link panda_link5: mass 0.1 -> 1.225946
- link panda_link5_sc: mass 0.1 -> None; geometry 
- link panda_link6: mass 0.1 -> 1.666555
- link panda_link6_sc: mass 0.1 -> None; geometry 
- link panda_link7: mass 0.1 -> 0.735522
- link panda_link7_sc: mass 0.1 -> None; geometry 
- link panda_rightfinger: mass 0.1 -> 0.015
Joints:
- added joint world_joint: type fixed, parent world, child panda_link0, origin xyz=0 0 0 rpy=0 0 0
