Commit message: - Corrigida a posição da nuvem de pontos no rviz

File: catkin_ws/src/panda_moveit_config/config/gazebo_panda_position_cleaned.urdf (robot description, URDF)
Before this commit: robot panda, 23 links, 22 joints
Joints:
- joint world_joint: origin xyz=0 0 0 rpy=0 0 0 -> xyz=-1.0 -0.6 1.02 rpy=0 0 -1.5708

Commit message: - Pick and place quase funcional. Braço se movimenta mas ainda não consegue fazer o pick

File: catkin_ws/src/panda_moveit_config/config/gazebo_panda_position_cleaned.urdf (robot description, URDF)
Before this commit: robot panda, 23 links, 22 joints
Joints:
- joint panda_finger_joint2: mimic joint=panda_finger_joint1 -> (none)
- joint world_joint: origin xyz=-1.0 -0.6 1.02 rpy=0 0 -1.5708 -> xyz=-1.0 -0.9 1.02 rpy=0 0 -1.5708
